File: OM345A/OM345A.kicad_sch (KiCad schematic)
At the start: 11 parts, among them J1 Conn_01x05, U1 MAR7+

Commit message: Added performance data
Other:
- note added: "Attenuation pad my be bypassed by zero Ohm R3 and R4 R5 not installed"
Changed lines of the file:
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@@
+		)
+	)
+	(text ""
+		(exclude_from_sim no)
+		(at 73.914 121.666 0)
+		(effects
+			(font
+				(size 2.54 2.54)
+			)
+		)
+	)
+	(text ""
+		(exclude_from_sim no)
+		(at 74.93 121.412 0)
+		(effects
+			(font
+				(size 12.954 12.954)
+			)
+		)
+	)
+	(text "Attenuation pad my be\nbypassed by zero Ohm R3\nand R4 R5 not installed"
+		(exclude_from_sim no)
+		(at 73.66 133.35 0)
+		(effects
+			(font
+				(size 2.54 2.54)
+			)
+		)
+	)
+	(text ""
+		(exclude_from_sim no)
+		(at 82.55 121.666 0)
+		(effects
+			(font
+				(size 2.54 2.54)
+			)
 		)
 	)
